Commit message: Add use_gripper arg to make gripper optional across launch files
Lets the arm/moveit/teleop launches build a bare-wrist URDF and SRDF
(no gripper links, joint, controller spawner, or mirroring) when no
gripper is physically installed, instead of always assuming one.

Co-Authored-By: Claude Sonnet 5 <noreply@anthropic.com>

File: i2rt_description/urdf/big_yam_linear_4310.urdf.xacro (robot description, xacro)
@@ -7,4 +7,9 @@
        instead of holding position - intended for a teleoperation leader arm. -->
   <xacro:arg name="compliant_mode" default="false"/>
+  <!-- false builds a bare-wrist arm: no gripper links/joint in the URDF and
+       no gripper_joint <ros2_control> block, for arms with no gripper
+       physically installed. See i2rt_teleop/launch/leader_follower.launch.py. -->
+  <xacro:arg name="use_gripper" default="true"/>
+  <xacro:property name="use_gripper" value="$(arg use_gripper)"/>
   <!-- Include big YAM arm and linear_4310 gripper macros -->
   <xacro:include filename="$(find i2rt_description)/urdf/big_yam_macro.xacro"/>
@@ -28,9 +33,11 @@
   </xacro:big_yam_arm>
   <!-- Instantiate linear_4310 gripper directly on the arm's wrist link -->
-  <xacro:gripper_linear_4310 prefix="" parent="link_6"/>
+  <xacro:if value="${use_gripper}">
+    <xacro:gripper_linear_4310 prefix="" parent="link_6"/>
+  </xacro:if>
   <!-- ros2_control hardware description (harmless when only visualizing —
        controller_manager only opens the CAN channel once this hardware
        component is actually loaded and activated) -->
   <xacro:big_yam_ros2_control prefix="" can_channel="$(arg can_channel)" use_mock_hardware="$(arg use_mock_hardware)"
-    compliant_mode="$(arg compliant_mode)"/>
+    compliant_mode="$(arg compliant_mode)" use_gripper="${use_gripper}"/>
 </robot>

File: i2rt_description/urdf/big_yam_ros2_control.xacro (robot description, xacro)
@@ -38,4 +38,8 @@
     motor of its own, so robot_state_publisher computes its transform from
     gripper_joint's published state without needing one.
+    use_gripper:=false omits this macro's gripper_joint <ros2_control> block
+    entirely (see big_yam_linear_4310.urdf.xacro, which also skips
+    instantiating the gripper_linear_4310 URDF macro in that case) - use for
+    an arm with no gripper physically installed. Defaults to true.
     gripper_joint (motor 7) DOES have an entry below: motor_id/motor_type/kp/kd
     are linear_4310.yml's real hardware defaults (DM4310, kp=20.0, kd=0.5).
@@ -85,5 +89,5 @@
   -->
   <xacro:macro name="big_yam_ros2_control"
-    params="prefix can_channel:=can0 use_mock_hardware:=false compliant_mode:=false">
+    params="prefix can_channel:=can0 use_mock_hardware:=false compliant_mode:=false use_gripper:=true">
     <ros2_control name="${prefix}big_yam_system" type="system">
       <hardware>
@@ -213,28 +217,30 @@
         <state_interface name="effort"/>
       </joint>
-      <joint name="${prefix}gripper_joint">
-        <param name="motor_id">7</param>
-        <param name="motor_type">DM4310</param>
-        <param name="kp">20.0</param>
-        <param name="kd">0.5</param>
-        <param name="direction">1.0</param>
-        <param name="offset">0.0</param>
-        <param name="gravity_comp_factor">0.0</param>
-        <param name="requires_calibration">true</param>
-        <!-- Verified against real hardware: the default polarity (1.0) paired
-             the raw hard-stops backwards; closed read back as open. -1.0
-             matches this gripper's actual motor wiring/rotation sense. -->
-        <param name="calibration_polarity">-1.0</param>
-        <param name="calibration_lower_limit_m">-0.0475</param>
-        <param name="calibration_upper_limit_m">0.0</param>
-        <command_interface name="position"/>
-        <command_interface name="velocity"/>
-        <command_interface name="effort"/>
-        <command_interface name="kp"/>
-        <command_interface name="kd"/>
-        <state_interface name="position"/>
-        <state_interface name="velocity"/>
-        <state_interface name="effort"/>
-      </joint>
+      <xacro:if value="${use_gripper}">
+        <joint name="${prefix}gripper_joint">
+          <param name="motor_id">7</param>
+          <param name="motor_type">DM4310</param>
+          <param name="kp">20.0</param>
+          <param name="kd">0.5</param>
+          <param name="direction">1.0</param>
+          <param name="offset">0.0</param>
+          <param name="gravity_comp_factor">0.0</param>
+          <param name="requires_calibration">true</param>
+          <!-- Verified against real hardware: the default polarity (1.0) paired
+               the raw hard-stops backwards; closed read back as open. -1.0
+               matches this gripper's actual motor wiring/rotation sense. -->
+          <param name="calibration_polarity">-1.0</param>
+          <param name="calibration_lower_limit_m">-0.0475</param>
+          <param name="calibration_upper_limit_m">0.0</param>
+          <command_interface name="position"/>
+          <command_interface name="velocity"/>
+          <command_interface name="effort"/>
+          <command_interface name="kp"/>
+          <command_interface name="kd"/>
+          <state_interface name="position"/>
+          <state_interface name="velocity"/>
+          <state_interface name="effort"/>
+        </joint>
+      </xacro:if>
     </ros2_control>
   </xacro:macro>
