Commit message: Add standard yam arm model, per-arm calibration registry, and fix gravity comp/gripper mass bugs
- Add full standard "yam" arm support (yam_macro.xacro, yam_ros2_control.xacro,
  yam_linear_4310.urdf.xacro, meshes) alongside the existing big_yam, following the
  same conventions. Hardware-verified direction and gravity_comp_factor calibration
  on multiple physical units of both arm models.
- Fix a real bug in YamSystemInterface: the internal diagnostics node (used for the
  gravity-comp KDL model) was constructed with an explicit namespace and subscribed
  to an absolute "/robot_description" topic, silently breaking gravity compensation
  whenever the hardware component ran under a ROS namespace (e.g. teleop's
  leader/follower launch). Fixed to inherit the real launch namespace.
- Fix link_6 (wrist-roll link) always carrying the linear_4310 gripper's housing
  mesh and ~0.55 kg mass even in bare-wrist (use_gripper:=false) mode, contradicting
  i2rt's own upstream reference models. Now conditional on use_gripper for both arm
  models; this also explains most of the apparent per-unit gravity_comp_factor
  variance found during teleop testing.
- Ramp gravity feed-forward torque alongside kp/kd on activation instead of applying
  it at full strength instantly, to avoid a real activation-time jump.
- Add a live-tunable gravity_comp_factor ROS parameter per joint for fast retuning
  without relaunching.
- Add i2rt_description/launch/arm_registry.py: a shared registry mapping an
  arbitrary arm name to its robot model, usual CAN channel, and validated per-unit
  parameter overrides, used via a new arm_name (leader_arm_name/follower_arm_name
  for teleop) argument across view_yam.launch.py, demo.launch.py, and
  leader_follower.launch.py.
- Add session_name support to leader_follower.launch.py for running multiple
  concurrent leader/follower sessions without node/topic/service collisions.
- Add i2rt_description/udev/99-i2rt-can.rules for persistent CAN interface naming
  by USB serial, independent of plug order.
- Correct the mirror_sign joint6 entry for mismatched leader/follower pairs (was
  wrongly flipped).
- Rewrite README.md to document the above; sweep the repo for stale comments left
  over from intermediate states during this work.

Co-Authored-By: Claude Sonnet 5 <noreply@anthropic.com>

File: i2rt_description/urdf/big_yam_macro.xacro (robot description, xacro)
@@ -10,5 +10,5 @@
     link), see gripper_linear_4310.xacro.
   -->
-  <xacro:macro name="big_yam_arm" params="prefix parent *origin">
+  <xacro:macro name="big_yam_arm" params="prefix parent use_gripper:=true *origin">
     <!-- Joint from parent to base_link -->
     <joint name="${prefix}base_joint" type="fixed">
@@ -207,29 +207,57 @@
       <limit lower="-2.0944" upper="2.0944" effort="10" velocity="10"/>
     </joint>
-    <!-- Link 6 / gripper housing. Visual/collision origin and inertial carried
-         over unchanged from yam_st_urdf_with_linear_gripper's own "gripper"
-         link (same frame convention as joint6 above), see comment there. -->
-    <link name="${prefix}link_6">
-      <visual>
-        <origin xyz="-0.014 -0.0463995 0.0731" rpy="0 0 0"/>
-        <geometry>
-          <mesh filename="package://i2rt_description/meshes/linear_4310/gripper.stl"/>
-        </geometry>
-        <material name="gripper_green">
-          <color rgba="0 0.4 0 1"/>
-        </material>
-      </visual>
-      <collision>
-        <origin xyz="-0.014 -0.0463995 0.0731" rpy="0 0 0"/>
-        <geometry>
-          <mesh filename="package://i2rt_description/meshes/linear_4310/gripper.stl"/>
-        </geometry>
-      </collision>
-      <inertial>
-        <origin xyz="-3.57066e-05 0.000249371 -0.0293133" rpy="0 0 0"/>
-        <mass value="0.553219"/>
-        <inertia ixx="0.000409668" ixy="5.44942e-07" ixz="7.91266e-07" iyy="0.000324942" iyz="-4.83958e-06" izz="0.000369249"/>
-      </inertial>
-    </link>
+    <!-- Link 6. use_gripper:=true: gripper housing - visual/collision origin
+         and inertial carried over unchanged from
+         yam_st_urdf_with_linear_gripper's own "gripper" link (same frame
+         convention as joint6 above), see comment there.
+         use_gripper:=false: this mesh+mass is NOT the bare arm's own
+         terminal link - it's entirely the GRIPPER's own housing, wrongly
+         baked into the base arm macro unconditionally before 2026-09-22.
+         Confirmed against i2rt-robotics/i2rt's own upstream reference
+         models: the arm-only MuJoCo model has joint6's body with NO <geom>
+         at all, and the upstream no_gripper.xml gripper-slot placeholder is
+         likewise meshless with a negligible mass (1e-6 kg) - gripper.stl
+         itself only exists under
+         i2rt/robot_models/gripper/linear_4310/assets/, i.e. it's the
+         gripper's asset, not the arm's - see yam_macro.xacro's matching
+         link_6 comment for the full evidence trail. Matches that convention
+         here: near-massless, mesh-less placeholder when no gripper is
+         attached, instead of always carrying the gripper housing's real
+         ~0.55 kg - this previously made every gravity_comp_factor value
+         tuned in use_gripper:=false mode compensate for phantom mass that
+         isn't actually there on real bare-wrist hardware. -->
+    <xacro:if value="${use_gripper}">
+      <link name="${prefix}link_6">
+        <visual>
+          <origin xyz="-0.014 -0.0463995 0.0731" rpy="0 0 0"/>
+          <geometry>
+            <mesh filename="package://i2rt_description/meshes/linear_4310/gripper.stl"/>
+          </geometry>
+          <material name="gripper_green">
+            <color rgba="0 0.4 0 1"/>
+          </material>
+        </visual>
+        <collision>
+          <origin xyz="-0.014 -0.0463995 0.0731" rpy="0 0 0"/>
+          <geometry>
+            <mesh filename="package://i2rt_description/meshes/linear_4310/gripper.stl"/>
+          </geometry>
+        </collision>
+        <inertial>
+          <origin xyz="-3.57066e-05 0.000249371 -0.0293133" rpy="0 0 0"/>
+          <mass value="0.553219"/>
+          <inertia ixx="0.000409668" ixy="5.44942e-07" ixz="7.91266e-07" iyy="0.000324942" iyz="-4.83958e-06" izz="0.000369249"/>
+        </inertial>
+      </link>
+    </xacro:if>
+    <xacro:unless value="${use_gripper}">
+      <link name="${prefix}link_6">
+        <inertial>
+          <origin xyz="0 0 0" rpy="0 0 0"/>
+          <mass value="1e-6"/>
+          <inertia ixx="1e-9" ixy="0" ixz="0" iyy="1e-9" iyz="0" izz="1e-9"/>
+        </inertial>
+      </link>
+    </xacro:unless>
     <!-- TCP Frame (Tool Center Point) -->
     <joint name="${prefix}tcp_joint" type="fixed">

File: i2rt_description/urdf/big_yam_ros2_control.xacro (robot description, xacro)
@@ -22,9 +22,42 @@
     values (which are +1 for both). Confirmed against real hardware: RViz
     showed joint4/6 rotating opposite the real arm before this fix.
-    gravity_comp_factor per joint is big_yam.yml's `gravity_comp_factor`
-    array — a per-joint scale on the KDL-computed gravity feed-forward torque
-    that YamSystemInterface adds every write() cycle (mirrors
+    gravity_comp_factor per joint below is NOT big_yam.yml's
+    `gravity_comp_factor` array ([1.0, 1.1, 1.0, 1.1, 1.0, 1.0]) - that
+    turned out not to be trustworthy as-is on real hardware, same as
+    yam_v1.yml's for the standard yam (see yam_ros2_control.xacro's header
+    comment for the full methodology this was re-tuned with). Current
+    status per joint: joint2/3/4 are tuned nonzero values from real hardware
+    (see each joint's own comment below), re-confirmed good after fixing
+    link_6's gripper-housing mesh/mass being wrongly present even in
+    bare-wrist (use_gripper:=false) mode (see yam_macro.xacro's link_6
+    comment for the full bug and evidence) - unlike the standard yam arm,
+    where that fix changed the bare-wrist mass model enough to require
+    re-tuning joints 2/3/4 (0.75/0.7/0.45 -> 0.9/0.9/0.95), this arm's
+    values held up as-is. joint1/joint6 are still 0.0, pending the same
+    re-tuning process; joint5 is 0.0 PERMANENTLY (see its own comment, not
+    pending). Each joint is a scale on the KDL-computed gravity feed-forward
+    torque that
+    YamSystemInterface adds every write() cycle (mirrors
     MotorChainRobot.update()'s `g * gravity_comp_factor` in the Python
-    reference). kp/kd are the URDF-fixed position-hold gains used whenever a
+    reference), and is live-tunable at runtime without relaunching via a
+    "gravity_comp_factor.<joint_name>" parameter on the hardware component's
+    internal diagnostics node (fully-qualified name
+    "/<prefix>big_yam_system_diagnostics" for a non-namespaced launch like
+    i2rt_moveit_config/demo.launch.py, or
+    "/<launch namespace>/<prefix>big_yam_system_diagnostics" under a
+    namespaced one like i2rt_teleop/leader_follower.launch.py - see
+    yam_system_interface.hpp's class comment, gravity compensation section,
+    for the exact usage and why the namespace behaves this way) - re-tune
+    joint by joint, tip-to-base (joint6 first,
+    joint1 last), with everything upstream of whichever joint is under test
+    physically braced/supported so each measurement is a clean, isolated
+    read rather than confounded by other joints still drooping freely; check
+    each joint's passive (fully unpowered, no control loop at all) behavior
+    first too, since at least one yam joint turned out to be dominated by
+    real mechanical friction that active comp only fought against rather
+    than helped - the same may or may not be true here. Once a value is
+    validated, write it back into this file as the new default (a live
+    `ros2 param set` change doesn't survive a relaunch on its own). kp/kd are
+    the URDF-fixed position-hold gains used whenever a
     controller doesn't claim the (also new) kp/kd command interfaces and
     compliant_mode is false — see YamSystemInterface's class comment for the
@@ -116,5 +149,13 @@
         <param name="kp">80.0</param>
         <param name="kd">5.0</param>
-        <param name="gravity_comp_factor">1.0</param>
+        <!-- Gravity comp intentionally left DISABLED (2026-09-22), not a
+             pending placeholder - decided not to re-tune this joint, so
+             leaving it at a known-safe, if unsupportive, 0.0 rather than
+             trusting big_yam.yml's never-independently-verified 1.0. If this
+             joint ever needs real gravity support, it should go through the
+             same live-tuned, braced-test methodology as joints 2/3/4 (see
+             this file's header comment), not just have big_yam.yml's value
+             restored blindly. -->
+        <param name="gravity_comp_factor">0.0</param>
         <param name="compliant_kd">0.5</param>
         <command_interface name="position"/>
@@ -134,5 +175,16 @@
         <param name="kp">80.0</param>
         <param name="kd">5.0</param>
-        <param name="gravity_comp_factor">1.1</param>
+        <!-- Validated on real hardware (2026-09-22), re-tuned live via the
+             gravity_comp_factor.joint2 parameter on diagnostics_node_ then
+             written back here - see this file's header comment for the
+             methodology. Not big_yam.yml's original 1.1: that value was
+             never independently verified for this arm either.
+             This is a SHARED file for every big_yam-model arm, not per-unit
+             - cross-checked on a second physical unit (same pattern as
+             yam_ros2_control.xacro's joint4): first unit wanted 1.0, second
+             wanted 0.975. Settled on 0.975 as the single shared value across
+             both. Re-confirmed good after fixing link_6's gripper-housing
+             mesh/mass bug (see this file's header comment). -->
+        <param name="gravity_comp_factor">0.975</param>
         <param name="compliant_kd">0.5</param>
         <command_interface name="position"/>
@@ -152,5 +204,14 @@
         <param name="kp">80.0</param>
         <param name="kd">5.0</param>
-        <param name="gravity_comp_factor">1.0</param>
+        <!-- Validated on real hardware (2026-09-22), re-tuned live via the
+             gravity_comp_factor.joint3 parameter on diagnostics_node_ then
+             written back here - see this file's header comment for the
+             methodology. Not big_yam.yml's original 1.0: that value was
+             never independently verified for this arm either. Cross-checked
+             on a second physical unit - transferred as-is, no per-unit
+             adjustment needed (unlike joint2). Re-confirmed good after
+             fixing link_6's gripper-housing mesh/mass bug (see this file's
+             header comment). -->
+        <param name="gravity_comp_factor">0.8</param>
         <param name="compliant_kd">0.5</param>
         <command_interface name="position"/>
@@ -170,5 +231,16 @@
         <param name="kp">40.0</param>
         <param name="kd">3.0</param>
-        <param name="gravity_comp_factor">1.1</param>
+        <!-- Validated on real hardware (2026-09-22), re-tuned live via the
+             gravity_comp_factor.joint4 parameter on diagnostics_node_ then
+             written back here - see this file's header comment for the
+             methodology. Not big_yam.yml's original 1.1: that value was
+             never independently verified for this arm either. Cross-checked
+             on a second physical unit - transferred as-is, no per-unit
+             adjustment needed (unlike joint2). Re-confirmed good after
+             fixing link_6's gripper-housing mesh/mass bug (see this file's
+             header comment) - despite the standard yam arm's equivalent
+             joint seeing the largest swing of its three after that same fix
+             (0.45->0.95), this arm's value held up as-is. -->
+        <param name="gravity_comp_factor">0.2</param>
         <param name="compliant_kd">0.3</param>
         <command_interface name="position"/>
@@ -188,5 +260,9 @@
         <param name="kp">40.0</param>
         <param name="kd">1.5</param>
-        <param name="gravity_comp_factor">1.0</param>
+        <!-- Validated on real hardware (2026-09-22): 0.0 is the correct,
+             PERMANENT value here, not a pending placeholder - see this
+             file's header comment for the methodology. Not
+             big_yam.yml's original 1.0. -->
+        <param name="gravity_comp_factor">0.0</param>
         <param name="compliant_kd">0.1</param>
         <command_interface name="position"/>
@@ -206,5 +282,7 @@
         <param name="kp">10.0</param>
         <param name="kd">1.5</param>
-        <param name="gravity_comp_factor">1.0</param>
+        <!-- Gravity comp DISABLED (2026-09-22) pending re-tuning, not
+             big_yam.yml's 1.0 - see this file's header comment for why. -->
+        <param name="gravity_comp_factor">0.0</param>
         <param name="compliant_kd">0.1</param>
         <command_interface name="position"/>

File: i2rt_description/urdf/gripper_linear_4310.xacro (robot description, xacro)
@@ -20,5 +20,5 @@
     <!-- Driving finger (right tip). Renamed from joint8 (source's gripper->
          tip_right) to match the single "gripper_joint" name expected by
-         yam_hardware_interface.py and joint_limits.yaml. -->
+         i2rt_hardware_interface/YamSystemInterface and joint_limits.yaml. -->
     <joint name="${prefix}gripper_joint" type="prismatic">
       <origin xyz="0.0226681 -0.0450619 -0.0545599" rpy="1.5708 0 0"/>

File: i2rt_description/urdf/yam_linear_4310.urdf.xacro (robot description, xacro)
@@ -3,5 +3,5 @@
   <xacro:arg name="can_channel" default="can0"/>
   <xacro:arg name="use_mock_hardware" default="false"/>
-  <!-- See big_yam_ros2_control.xacro's macro comment: true makes this arm
+  <!-- See yam_ros2_control.xacro's macro comment: true makes this arm
        hand-backdrivable (kp=0, kd=each joint's "compliant_kd" <param>)
        instead of holding position - intended for a teleoperation leader arm. -->
@@ -12,8 +12,8 @@
   <xacro:arg name="use_gripper" default="true"/>
   <xacro:property name="use_gripper" value="$(arg use_gripper)"/>
-  <!-- Include big YAM arm and linear_4310 gripper macros -->
-  <xacro:include filename="$(find i2rt_description)/urdf/big_yam_macro.xacro"/>
+  <!-- Include standard yam arm and linear_4310 gripper macros -->
+  <xacro:include filename="$(find i2rt_description)/urdf/yam_macro.xacro"/>
   <xacro:include filename="$(find i2rt_description)/urdf/gripper_linear_4310.xacro"/>
-  <xacro:include filename="$(find i2rt_description)/urdf/big_yam_ros2_control.xacro"/>
+  <xacro:include filename="$(find i2rt_description)/urdf/yam_ros2_control.xacro"/>
   <!-- Materials -->
   <material name="orange">
@@ -28,8 +28,8 @@
   <!-- World link (fixed base) -->
   <link name="world"/>
-  <!-- Instantiate big YAM arm -->
-  <xacro:big_yam_arm prefix="" parent="world" use_gripper="${use_gripper}">
+  <!-- Instantiate yam arm -->
+  <xacro:yam_arm prefix="" parent="world" use_gripper="${use_gripper}">
     <origin xyz="0 0 0" rpy="0 0 0"/>
-  </xacro:big_yam_arm>
+  </xacro:yam_arm>
   <!-- Instantiate linear_4310 gripper directly on the arm's wrist link -->
   <xacro:if value="${use_gripper}">
@@ -39,5 +39,5 @@
        controller_manager only opens the CAN channel once this hardware
        component is actually loaded and activated) -->
-  <xacro:big_yam_ros2_control prefix="" can_channel="$(arg can_channel)" use_mock_hardware="$(arg use_mock_hardware)"
+  <xacro:yam_ros2_control prefix="" can_channel="$(arg can_channel)" use_mock_hardware="$(arg use_mock_hardware)"
     compliant_mode="$(arg compliant_mode)" use_gripper="${use_gripper}"/>
 </robot>
